File: Board.sch (EAGLE design)
At the start: 24 parts

Commit message: premilinary rev 2, fixed Ac/DC footprint, removed on-board switch and added mains outputs
Parts:
- removed MAINS-IN: (no value), pinhead:PINHD-1X3
- removed SWITCH: (no value), pinhead:PINHD-1X2
- R11, R12, R9: device rcl:R-US_R0805 -> rcl:R-US_R0603
- renumbered RAC05-05SK to RAC05-K
Connections:
- removed net N$7: MAINS-IN.3, SWITCH.1
- removed net PGND: MAINS-IN.1
- net VAC(L)-INPUT: no longer SWITCH.2
- net VAC(N): no longer MAINS-IN.2
Other:
- moved on the sheet: F1
Changed lines of the file:
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@@
 <parts>
 <part name="STM32F070F6" library="SousVide Library" deviceset="STM32F07" device="" value=""/>
-<part name="RAC05-05SK" library="SousVide Library" deviceset="AC/DC-CONVERTER" device=""/>
 <part name="+3V1" library="supply1" library_urn="urn:adsk.eagle:library:371" deviceset="+3V3" device=""/>
 <part name="SUPPLY1" library="supply2" library_urn="urn:adsk.eagle:library:372" deviceset="PE" device=""/>
@@
 <part name="R5" library="rcl" library_urn="urn:adsk.eagle:library:334" deviceset="R-US_" device="R0603" package3d_urn="urn:adsk.eagle:package:23555/2" value="1k5"/>
 <part name="THERMISTOR" library="pinhead" library_urn="urn:adsk.eagle:library:325" deviceset="PINHD-1X2" device="" package3d_urn="urn:adsk.eagle:package:22435/2"/>
-<part name="MAINS-IN" library="pinhead" library_urn="urn:adsk.eagle:library:325" deviceset="PINHD-1X3" device="" package3d_urn="urn:adsk.eagle:package:22458/2"/>
-<part name="SWITCH" library="pinhead" library_urn="urn:adsk.eagle:library:325" deviceset="PINHD-1X2" device="" package3d_urn="urn:adsk.eagle:package:22435/2"/>
-<part name="R9" library="rcl" library_urn="urn:adsk.eagle:library:334" deviceset="R-US_" device="R0805" package3d_urn="urn:adsk.eagle:package:23553/2" value="250"/>
-<part name="R11" library="rcl" library_urn="urn:adsk.eagle:library:334" deviceset="R-US_" device="R0805" package3d_urn="urn:adsk.eagle:package:23553/2" value="250"/>
-<part name="R12" library="rcl" library_urn="urn:adsk.eagle:library:334" deviceset="R-US_" device="R0805" package3d_urn="urn:adsk.eagle:package:23553/2" value="250"/>
+<part name="R9" library="rcl" library_urn="urn:adsk.eagle:library:334" deviceset="R-US_" device="R0603" package3d_urn="urn:adsk.eagle:package:23555/2" value="250"/>
+<part name="R11" library="rcl" library_urn="urn:adsk.eagle:library:334" deviceset="R-US_" device="R0603" package3d_urn="urn:adsk.eagle:package:23555/2" value="250"/>
+<part name="R12" library="rcl" library_urn="urn:adsk.eagle:library:334" deviceset="R-US_" device="R0603" package3d_urn="urn:adsk.eagle:package:23555/2" value="250"/>
 <part name="SV2" library="con-lstb" library_urn="urn:adsk.eagle:library:162" deviceset="MA06-1" device="" package3d_urn="urn:adsk.eagle:package:8340/1"/>
 <part name="PE6" library="YabzLib" deviceset="GND" device=""/>
@@
 <part name="JP7" library="pinhead" library_urn="urn:adsk.eagle:library:325" deviceset="PINHD-1X3" device="" package3d_urn="urn:adsk.eagle:package:22458/2"/>
 <part name="JP8" library="pinhead" library_urn="urn:adsk.eagle:library:325" deviceset="PINHD-1X3" device="" package3d_urn="urn:adsk.eagle:package:22458/2"/>
+<part name="RAC05-K" library="SousVide Library" deviceset="AC/DC-CONVERTER" device=""/>
 </parts>
 <sheets>
@@
 <instances>
 <instance part="STM32F070F6" gate="G$1" x="-30.48" y="81.28"/>
-<instance part="RAC05-05SK" gate="G$1" x="81.28" y="88.9"/>
 <instance part="+3V1" gate="G$1" x="137.16" y="99.06"/>
 <instance part="SUPPLY1" gate="PE" x="101.6" y="78.74" smashed="yes"/>
@@
 <instance part="+3V3" gate="G$1" x="0" y="88.9"/>
 <instance part="SUPPLY4" gate="PE" x="0" y="76.2" smashed="yes"/>
-<instance part="F1" gate="G$1" x="50.8" y="93.98"/>
+<instance part="F1" gate="G$1" x="53.34" y="93.98"/>
 <instance part="SUPPLY5" gate="PE" x="-58.42" y="88.9" smashed="yes"/>
-<instance part="U$1" gate="G$1" x="35.56" y="68.58"/>
+<instance part="U$1" gate="G$1" x="43.18" y="68.58"/>
 <instance part="R3" gate="G$1" x="45.72" y="48.26" smashed="yes" rot="R270">
 <attribute name="NAME" x="47.2186" y="46.99" size="1.778" layer="95" rot="R270"/>
@@
 </instance>
 <instance part="THERMISTOR" gate="G$1" x="121.92" y="-25.4"/>
-<instance part="MAINS-IN" gate="A" x="27.94" y="76.2" rot="R180"/>
-<instance part="SWITCH" gate="G$1" x="27.94" y="88.9" rot="R180"/>
 <instance part="R9" gate="G$1" x="-38.1" y="38.1" rot="R180"/>
 <instance part="R11" gate="G$1" x="-38.1" y="22.86" rot="R180"/>
@@
 <instance part="JP7" gate="A" x="88.9" y="15.24" rot="R180"/>
 <instance part="JP8" gate="A" x="116.84" y="15.24" rot="R180"/>
+<instance part="RAC05-K" gate="G$1" x="81.28" y="88.9"/>
 </instances>
 <busses>
@@
 <wire x1="109.22" y1="91.44" x2="109.22" y2="93.98" width="0.1524" layer="91"/>
 <junction x="109.22" y="93.98"/>
-<pinref part="RAC05-05SK" gate="G$1" pin="VOUT+"/>
 <wire x1="96.52" y1="93.98" x2="109.22" y2="93.98" width="0.1524" layer="91"/>
+<pinref part="RAC05-K" gate="G$1" pin="VOUT+"/>
 </segment>
 <segment>
@@
 <net name="PE" class="0">
 <segment>
-<pinref part="RAC05-05SK" gate="G$1" pin="VOUT-"/>
 <wire x1="96.52" y1="83.82" x2="101.6" y2="83.82" width="0.1524" layer="91"/>
 <wire x1="101.6" y1="83.82" x2="101.6" y2="81.28" width="0.1524" layer="91"/>
 <pinref part="SUPPLY1" gate="PE" pin="PE"/>
+<pinref part="RAC05-K" gate="G$1" pin="VOUT-"/>
 </segment>
 <segment>
@@
 <net name="VAC(L)" class="0">
 <segment>
-<pinref part="RAC05-05SK" gate="G$1" pin="AC(L)"/>
 <wire x1="66.04" y1="93.98" x2="60.96" y2="93.98" width="0.1524" layer="91"/>
 <wire x1="60.96" y1="93.98" x2="60.96" y2="96.52" width="0.1524" layer="91"/>
 <label x="65.024" y="98.552" size="1.778" layer="95" rot="R180"/>
 <pinref part="F1" gate="G$1" pin="2"/>
-<wire x1="55.88" y1="93.98" x2="60.96" y2="93.98" width="0.1524" layer="91"/>
+<wire x1="58.42" y1="93.98" x2="60.96" y2="93.98" width="0.1524" layer="91"/>
 <junction x="60.96" y="93.98"/>
+<pinref part="RAC05-K" gate="G$1" pin="AC(L)"/>
 </segment>
 </net>
 <net name="VAC(N)" class="0">
 <segment>
-<pinref part="RAC05-05SK" gate="G$1" pin="AC(N)"/>
-<wire x1="30.48" y1="76.2" x2="43.18" y2="76.2" width="0.1524" layer="91"/>
-<wire x1="43.18" y1="76.2" x2="43.18" y2="83.82" width="0.1524" layer="91"/>
-<wire x1="43.18" y1="83.82" x2="45.72" y2="83.82" width="0.1524" layer="91"/>
-<wire x1="45.72" y1="83.82" x2="66.04" y2="83.82" width="0.1524" layer="91"/>
-<wire x1="45.72" y1="83.82" x2="45.72" y2="86.36" width="0.1524" layer="91"/>
-<label x="43.18" y="86.36" size="1.778" layer="95"/>
-<junction x="45.72" y="83.82"/>
-<pinref part="MAINS-IN" gate="A" pin="2"/>
+<wire x1="35.56" y1="83.82" x2="66.04" y2="83.82" width="0.1524" layer="91"/>
+<pinref part="RAC05-K" gate="G$1" pin="AC(N)"/>
+<label x="35.56" y="83.82" size="1.778" layer="95" rot="R180"/>
 </segment>
 </net>
@@
 <segment>
 <pinref part="F1" gate="G$1" pin="1"/>
-<pinref part="SWITCH" gate="G$1" pin="2"/>
-<wire x1="35.56" y1="93.98" x2="43.18" y2="93.98" width="0.1524" layer="91"/>
-<wire x1="30.48" y1="88.9" x2="35.56" y2="88.9" width="0.1524" layer="91"/>
-<wire x1="35.56" y1="88.9" x2="35.56" y2="93.98" width="0.1524" layer="91"/>
-</segment>
-</net>
-<net name="PGND" class="0">
-<segment>
-<wire x1="30.48" y1="73.66" x2="35.56" y2="73.66" width="0.1524" layer="91"/>
-<wire x1="35.56" y1="73.66" x2="35.56" y2="71.12" width="0.1524" layer="91"/>
+<wire x1="40.64" y1="93.98" x2="45.72" y2="93.98" width="0.1524" layer="91"/>
+<label x="40.64" y="93.98" size="1.778" layer="95" rot="R180"/>
+</segment>
+</net>
+<net name="VAC(G)" class="0">
+<segment>
+<wire x1="35.56" y1="76.2" x2="43.18" y2="76.2" width="0.1524" layer="91"/>
+<wire x1="43.18" y1="76.2" x2="43.18" y2="71.12" width="0.1524" layer="91"/>
 <pinref part="U$1" gate="G$1" pin="PE"/>
-<pinref part="MAINS-IN" gate="A" pin="1"/>
+<label x="35.56" y="76.2" size="1.778" layer="95" rot="R180"/>
 </segment>
 </net>
@@
 </segment>
 </net>
-<net name="N$7" class="0">
-<segment>
-<pinref part="MAINS-IN" gate="A" pin="3"/>
-<wire x1="30.48" y1="78.74" x2="35.56" y2="78.74" width="0.1524" layer="91"/>
-<wire x1="35.56" y1="78.74" x2="35.56" y2="86.36" width="0.1524" layer="91"/>
-<pinref part="SWITCH" gate="G$1" pin="1"/>
-<wire x1="35.56" y1="86.36" x2="30.48" y2="86.36" width="0.1524" layer="91"/>
-</segment>
-</net>

Commit message: added DC power LEDs
Parts:
- added D1, D2: (no value), SparkFun-LED:LED0603
- added R1, R6: 250, rcl:R-US_R0603
Connections:
- removed net PE: C1.2, C2.2, JP1.4, JP2.3, JP4.3, JP5.3, JP6.3, JP7.3, JP8.3, LM117.ADJ, R5.2, RAC05-K.VOUT-, STM32F070F6.BOOT0, STM32F070F6.VSS
- new net N$1: D1.C, R1.1
- new net N$2: D2.C, R6.1
- net +3V3: now also D1.A
- net +5V: now also D2.A
- net GND: now also C1.2, C2.2, JP1.4, JP2.3, JP4.3, JP5.3, JP6.3, JP7.3, JP8.3, LM117.ADJ, R1.2, R5.2, R6.2, RAC05-K.VOUT-, STM32F070F6.BOOT0, STM32F070F6.VSS
