File: PCB/Board.sch (EAGLE design)
At the start: 32 parts, among them K1 G5LE, K2 G5LE, K3 G5LE, Q1 MOSFET-NCHANNELSMD, Q2 MOSFET-NCHANNELSMD, Q3 MOSFET-NCHANNELSMD

Commit message: v2
Parts:
- removed D3, D4, D5: 1N4004, diode:1N4004
- removed K1, K2, K3: G5LE, relay:G5LE
- removed Q2, Q3: MOSFET-NCHANNELSMD, fets:MOSFET-NCHANNELSMD
- removed RAC05-K: AC/DC-CONVERTER, SousVide Library:AC/DC-CONVERTER
- removed SV2: (no value), con-lstb:MA06-1
- added C10, C5, C8: 1u, rcl:C-USC0603
- added C11, C9: 2.2uF, rcl:C-USC0603
- added C3, C4: 0.1u, rcl:C-USC0603
- added C6: 10u, rcl:C-USC0603
- added C7: 44u, rcl:C-USC0603
- added D7: 1N4148DO35-7, diode:1N4148DO35-7
- added J1, J6: (no value), SparkFun-Connectors:CONN_04
- added J2, J3, J4, J5: (no value), Wurth_Elektronik_Electromechanic_Wire_to_Board_Connectors_rev19a:66100211622
- added L1: 40Ohm@100MHz, Wurth_EMC Components_WE-CBF:WE-CBF_0805_74279208_WB_HS
- added LED1, LED2, LED3, LED4: Yellow, SparkFun-LED:LED-YELLOW0603
- added OK1, OK2, OK3, OK4: MOC3031S, optocoupler:MOC3031S
- added OK5: 4N35, optocoupler:4N35
- added PS1: RAC03-05SK, SousVide Library:RAC03-05SK
- added R13, R19, R23, R27: 2k, rcl:R-US_R0603
- added R14: 1k5, rcl:R-US_R0603
- added R15, R20, R28: 250, rcl:R-US_R0603
- added R16, R21, R25, R29, R36, R37: 1k, rcl:R-US_R0603
- added R17: P594, varistor:P594
- added R18, R22, R26: 500r, rcl:R-US_R0603
- added R24: 24k, rcl:R-US_R0603
- added R30: 5k, rcl:R-US_R0603
- added R31: 10k, rcl:R-US_R0603
- added R32: 100k, rcl:R-US_R0603
- added R33: 330r, rcl:R-US_R0603
- added R34, R35: 50k, rcl:R-US_R0603
- added SV1: (no value), con-lstb:MA05-1
- added T1, T2, T3, T4: (no value), transistor:-NPN-SOT23-EBC
- added U$1: MDB8S, SousVide Library:MDB8S
- added U$3, U$4, U$5, U$6: SST04K-800SW, SousVide Library:SST04K-800SW
- added X1: B3P-VH, con-JST VH:B3P-VH
- Q1: value MOSFET-NCHANNELSMD -> BC847SMD; device fets:MOSFET-NCHANNELSMD -> SousVide Library:BC847SMD
- R10: value 250 -> 500r
- R2: value 3k3 -> 10k
- R7: value 250 -> 10k
- R8: value 250 -> 1k5
Connections:
- removed net GND: C1.2, C2.2, JP1.4, LM117.ADJ, R1.2, R5.2, R6.2, RAC05-K.VOUT-, STM32F070F6.BOOT0, STM32F070F6.VSS, SV2.4
- removed net N$6: D5.A, K31.2, Q2.D
- removed net RELAY1: R7.2, STM32F070F6.PA0
- removed net RELAY2: R8.2, STM32F070F6.PA3
- removed net RELAY3: R10.2, STM32F070F6.PA5
- removed net SWO: SV2.1
- removed net VAC(L): F1.2, K12.S, K22.S, K32.S, RAC05-K.AC(L)
- removed net VAC(L)-OUTPUT1: K12.P
- removed net VAC(L)-OUTPUT2: K32.P
- removed net VAC(L)-OUTPUT3: K22.P
- removed net VAC(N): RAC05-K.AC(N)
- new net CTRL1: R18.2, STM32F070F6.PA3
- new net CTRL2: R22.2, STM32F070F6.PA2
- new net CTRL3: R26.2, STM32F070F6.PA1
- new net CTRL4: R10.2, STM32F070F6.PA0
- new net ENCODER_A: R36.2, STM32F070F6.PA6, SV1.5
- new net ENCODER_B: R37.2, STM32F070F6.PA5, SV1.4
- new net ENCODER_BUTTON: STM32F070F6.PA4, SV1.3
- new net FET4: R26.1, T4.B
- new net N$10: LED1.A, R16.2
- new net N$11: J3.1, U$3.A2
- new net N$12: OK2.A, R19.1
- new net N$13: OK2.A1, R20.2
- new net N$14: R20.1, U$4.G
- new net N$15: LED2.A, R21.2
- new net N$16: J2.1, U$4.A2
- new net N$17: LED3.C, OK3.C, T3.C
- new net N$18: OK3.A, R23.1
- new net N$20: OK3.A1, R24.2
- new net N$23: R24.1, U$5.G
- new net N$24: LED3.A, R25.2
- new net N$25: J4.1, U$5.A2
- new net N$26: LED4.C, OK4.C, T4.C
- new net N$27: OK4.A, R27.1
- new net N$28: OK4.A1, R28.2
- new net N$29: R28.1, U$6.G
- new net N$30: LED4.A, R29.2
- new net N$31: J5.1, U$6.A2
- new net N$32: D7.C, Q1.B, R30.2, U$1.-
- new net N$33: C7.1, R30.1, R33.1, U$1.+
- new net N$34: C7.2, D7.A, Q1.E
- new net N$35: OK5.C, Q1.C
- new net N$36: OK5.BAS, R32.1
- new net N$37: OK5.A, R33.2
- new net N$38: R34.2, U$1.AC1
- new net N$39: R35.2, U$1.AC2
- new net N$43: R2.2, STM32F070F6.BOOT0
- new net N$5: LED1.C, OK1.C, T1.C
- new net N$7: OK1.A1, R15.2
- new net N$8: OK1.A, R13.1
- new net N$9: R15.1, U$3.G
- new net THERM-CALIBRATE: R14.2, R8.1, STM32F070F6.PA7
- new net V+: F1.2, J2.2, J3.2, J4.2, J5.2, OK1.A2, OK2.A2, OK3.A2, OK4.A2, PS1.VAC_IN(L), R17.2, R34.1
- new net V-: PS1.VAC_IN(N), R17.1, R35.1, U$3.A1, U$4.A1, U$5.A1, U$6.A1, X1.2
- new net ZERO-CROSS-DETECT: OK5.COL, R31.2
- net +3V3: now also C10.1, C11.1, C4.1, C5.1, C9.1, J6.4, L1.1, R14.1, R31.1, R36.1, R37.1, R7.1, SV1.2; no longer R2.2, STM32F070F6.VDDA, SV2.6
- net +5V: now also C6.1, PS1.+VOUT, R13.2, R16.1, R19.2, R21.1, R23.2, R25.1, R27.2, R29.1; no longer D3.C, D4.C, D5.C, K11.1, K21.1, K31.1, RAC05-K.VOUT+
- net FET1: now also R18.1, T2.B; no longer Q1.G, R7.1
- net FET2: now also R22.1, T3.B; no longer Q2.G, R8.1
- net FET3: now also T1.B; no longer Q3.G
- net N$19: now also J1.4; no longer SV2.5
- net N$21: now also J1.2; no longer SV2.3
- net N$22: now also J1.1; no longer SV2.2
- net N$3: now also C3.1, C8.1, L1.2, STM32F070F6.VDDA; no longer D4.A, K11.2, Q1.D
- net N$4: now also LED2.C, OK2.C, T2.C; no longer D3.A, K21.2, Q3.D
- net NRST: now also R7.2; no longer R2.1
- net PE: now also C1.2, C10.2, C11.2, C2.2, C3.2, C4.2, C5.2, C6.2, C8.2, C9.2, J1.3, J6.3, JP1.4, LM117.ADJ, OK5.EMI, PS1.-VOUT, R1.2, R2.1, R32.2, R5.2, R6.2, R8.2, STM32F070F6.VSS, SV1.1, T1.E, T2.E, T3.E, T4.E, X1.1; no longer Q1.S, Q2.S, Q3.S
- net RX: now also J6.2
- net TX: now also J6.1
- net VAC(L)-INPUT: now also X1.3
Other:
- moved on the sheet: C1, C2, D1, D2, F1, LM117, R1, R10, R11, R12, R2, R5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

Commit message: started v4 redesign
Parts:
- removed R11, R12, R28, R9: 250, rcl:R-US_R0603
- removed R24: 24k, rcl:R-US_R0603
- R14, R8: value 1k5 -> (none); device rcl:R-US_R0603 -> rcl:R-US_0613/15
- R15, R20: value 250 -> (none); device rcl:R-US_R0603 -> rcl:R-US_0613/15
Connections:
- removed net N$19: J1.4, R9.2
- removed net N$21: J1.2, R11.2
- removed net N$22: J1.1, R12.2
- removed net THERM-CALIBRATE: R14.2, R8.1, STM32F070F6.PA7
- net +3V3: no longer R14.1
- net ENCODER_A: now also STM32F070F6.PA5; no longer STM32F070F6.PA6
- net ENCODER_B: now also STM32F070F6.PA6; no longer STM32F070F6.PA5
- net ENCODER_BUTTON: now also STM32F070F6.PA7; no longer STM32F070F6.PA4
- net N$13: now also R8.1; no longer R20.2
- net N$14: now also R8.2; no longer R20.1
- net N$20: now also R15.1; no longer R24.2
- net N$23: now also R15.2; no longer R24.1
- net N$28: now also R14.1; no longer R28.2
- net N$29: now also R14.2; no longer R28.1
- net N$7: now also R20.1; no longer R15.2
- net N$9: now also R20.2; no longer R15.1
- net NRST: now also J1.1; no longer R12.1
- net PE: no longer R8.2
- net SWCLK: now also J1.4; no longer R9.1
- net SWDIO: now also J1.2; no longer R11.1
- net ZERO-CROSS-DETECT: now also STM32F070F6.PA4
Other:
- moved on the sheet: R14, R15, R20, R8
